Commit message: walking morphLynX (biped)

File: rsc/morphLynX/morphLynX.urdf (robot description, URDF)
Before this commit: robot p4, 42 links, 41 joints
Links:
- link CAMERA-L: mass 0.00441438009619701 -> 0.00441437949580177
- link CAMERA-R: mass 0.00441438279557042 -> 0.00441438009619701
- link FRONT-CAPLING: mass 0.00270228717508012 -> 0.00270228717508013
- link L-FOOT: mass 0.00920518287932567 -> 0.00920518287932568
- link L-LINK-HIP-ANKLE: mass 0.0128808114115962 -> 0.00969881141159618
- link L-LINK-TIBIA-FOOT: mass 0.00862384221571941 -> 0.00862384221571942
- link L-SC-FOOT-PITCH: mass 0.00307410332930239 -> 0.00307410332930238
- link L-SC-HIP-ROLL: mass 0.00388168562397068 -> 0.00388168562397067
- link L-SC2-FOOT-PITCH: mass 0.00563001173416682 -> 0.00563001173416683
- link L-SERVO-ANKLE: mass 0.00691519232272843 -> 0.00691519224850052
- link L-SERVO-FOOT-PITCH: mass 0.00691519226285069 -> 0.0069151922968296
- link L-SERVO-FOOT-ROLL: mass 0.00691519440391438 -> 0.00691519441607537
- link L-SERVO-HIP-PITCH: mass 0.00691519228445372 -> 0.00691519226383927
- link L-SERVO-HIP-ROLL: mass 0.00691519223632289 -> 0.00691519221564618
- link L-SERVO-TIBIA-PITCH: mass 0.00691519226322913 -> 0.0069151922750263
- link L-SUCTION: mass 0.007293938189965 -> 0.00729393814141169
- link R-FOOT: mass 0.00920518301651191 -> 0.00920518301651192
- link R-LINK-HIP-ANKLE: mass 0.0128808114115962 -> 0.00969881141159618
- link R-LINK-TIBIA-FOOT: mass 0.00862384221571939 -> 0.0086238422157194
- link R-SC-HIP-PITCH: mass 0.00388168562397067 -> 0.00388168562397068
- link R-SERVO-ANKLE-PITCH: mass 0.00691519224247509 -> 0.00691519221533839
- link R-SERVO-FOOT-PITCH: mass 0.00691519225207978 -> 0.00691519223321423
- link R-SERVO-FOOT-ROLL: mass 0.00691519435513484 -> 0.00691519435951329
- link R-SERVO-HIP-PITCH: mass 0.00691519223490345 -> 0.00691519224700007
- link R-SERVO-HIP-ROLL: mass 0.00691519222535946 -> 0.00691519223713882
- link R-SERVO-TIBIA-PITCH: mass 0.00691519223380914 -> 0.00691519221947937
- link R-SUCTION: mass 0.00729393814209891 -> 0.00729393816571459
- link SERVO-FRONT-CAPLING-PITCH: mass 0.00691519224201597 -> 0.00691519225617411
- link SERVO-REAR-CAPLING-ROLL: mass 0.00691519222019108 -> 0.00691519224449398
Joints:
- joint CAMERA-L: origin xyz=0.00995593171266154 0.038 0.0133 rpy=1.5707963267949 0 -1.5707963267949 -> xyz=0.00420593171264967 0.0402999999999998 0.00525000000003185 rpy=0 0 0
- joint CAMERA-R: origin xyz=0.00995593171266154 -0.038 0.0133 rpy=1.5707963267949 0 -1.5707963267949 -> xyz=0.00420593171264593 -0.0357000000000002 0.00525000000003465 rpy=0 0 0
- joint CAPLING-F-PITCH: origin xyz=0 0 0 rpy=0 0.00136062510321918 -3.14159264419998 -> xyz=-0.00525000000000001 0 0 rpy=0 0.00136062510321918 -3.14159264419998; type continuous -> revolute
- joint CAPLING-REAR-ROLL: type continuous -> revolute
- joint CONTROL-BOX: origin xyz=-0.0020940682873385 0 0.005 rpy=0 0 0 -> xyz=-0.00209406828734438 0 0.00500000000002512 rpy=0 0 3.14159265358978
- joint L-ANKLE-PITCH: limit lower=-6.28 upper=6.28 effort=80 velocity=15 -> lower=-4.4 upper=0.25 effort=80 velocity=15; type continuous -> revolute
- joint L-FOOT: origin xyz=0.00525000000000002 -0.0236702854642496 0 rpy=1.57079632678999 0 3.14159265358979 -> xyz=0.00839734742823202 -0.0239671534725504 -0.00264083015807315 rpy=0 -0.510525281997019 -1.57079632283259
- joint L-FOOT-PITCH: limit lower=-6.28 upper=6.28 effort=80 velocity=15 -> lower=-1.1 upper=3.05 effort=80 velocity=15; origin xyz=-0.0691703472599892 0.000991343468366913 0.00492086078353873 rpy=3.14159265358964 0.986473163636373 -3.14159265358979 -> xyz=-0.070999999999994 0.000991343468367011 0 rpy=3.14159265358964 0.986473163636372 -3.14159265358979; type continuous -> revolute
- joint L-FOOT-ROLL: origin xyz=-0.0336297145357536 0 0.00550865653160941 rpy=-3.14159265358953 -1.568123927556 1.57079632679464 -> xyz=-0.028379714535749 0 0.00649999999997644 rpy=-3.14159265358953 -1.568123927556 1.57079632679464; type continuous -> revolute
- joint L-HIP-PITCH: limit lower=-6.28 upper=6.28 effort=80 velocity=15 -> lower=-0.6 upper=2.55 effort=80 velocity=15; origin xyz=-0.00525000000000002 0 0 rpy=-3.1415926535897 0.494565195779334 3.14159265358968 -> xyz=-0.00525000000000001 0 0 rpy=-3.1415926535897 0.494565195779334 3.14159265358968; type continuous -> revolute
- joint L-HIP-ROLL: limit lower=-6.28 upper=6.28 effort=80 velocity=15 -> lower=-3.15 upper=1.4 effort=80 velocity=15; origin xyz=0 0.011 0 rpy=3.14159265358725 -1.56867970079681 -3.14159265358726 -> xyz=-0.00525000000000006 0.0287557291019455 0 rpy=3.14159265358725 -1.56867970079681 -3.14159265358726; type continuous -> revolute
- joint L-LINK-ANKLE-TIBIA: origin xyz=0.08225 -0.000999999999994901 0 rpy=1.5707963267949 0 -3.14159265358979 -> xyz=0.08225 -0.000999999999994859 0 rpy=1.5707963267949 0 -3.14159265358979
- joint L-SC-FOOT-PITCH: origin xyz=0 0.01 0 rpy=1.5707963267949 0 -3.14159265358979 -> xyz=0.00524999999999309 0.0105086565316094 0 rpy=1.5707963267949 0 -3.14159265358979
- joint L-SC-HIP-ROLL: origin xyz=0.00995593171266153 0.038 -0.0083 rpy=1.5707963267949 0 -1.5707963267949 -> xyz=0.0099559317126789 0.0379999999999999 -0.00829999999998628 rpy=1.5707963267949 0 -1.57079632679491
- joint L-SC2-FOOT-PITCH: origin xyz=0 0 0 rpy=1.5707963267949 0 3.14159265358979 -> xyz=0.00524999999998904 -0.000991343468366976 0 rpy=1.5707963267949 0 3.14159265358979
- joint L-SERVO-HIP-PITCH: origin xyz=0.00551111227819222 0.0261000000000001 -0.00555001176027257 rpy=1.5707963267949 0 -3.14159265358978 -> xyz=0.00549999999999939 0.00834427089805467 -0.0107999999999998 rpy=1.5707963267949 0 -3.14159265358978
- joint L-SUCTION: origin xyz=-0.03092034725999 -0.00780000000000004 0.00492086078353519 rpy=3.14159265358979 0 -3.14159265358979 -> xyz=-0.0327499999999984 -0.00779999999999992 0 rpy=3.14159265358979 0 -3.14159265358979
- joint L-SUCTIONCUP: origin xyz=0 -0.0116636317567518 -0.00454575689715984 rpy=1.06027104479611 0 -3.14159265094917 -> xyz=-0.000701757848402165 -0.00314734742580583 -0.00994844417065108 rpy=0 0 1.57079632333783
- joint L-TIBIA-PITCH: limit lower=-6.28 upper=6.28 effort=80 velocity=15 -> lower=-0.2 upper=3.7 effort=80 velocity=15; origin xyz=0 0 0 rpy=3.14159265358979 -1.21482038941994 -3.14159265358979 -> xyz=-0.00525000000000003 0 0 rpy=3.14159265358979 -1.21482038941994 -3.14159265358979; type continuous -> revolute
- joint R-ANKLE-PITCH: limit lower=-6.28 upper=6.28 effort=80 velocity=15 -> lower=-0.25 upper=4.4 effort=80 velocity=15; origin xyz=0.0710000000000002 0 0 rpy=0 0.802849328179599 -3.14159265358979 -> xyz=0.0710000000000001 0 0 rpy=0 0.802849328179599 -3.14159265358979; type continuous -> revolute
- joint R-FOOT: origin xyz=0.00525000000000002 -0.0237019612288078 0 rpy=-1.5707963267949 0 0 -> xyz=0.00210265257176806 -0.0239988292371081 0.00264083015806924 rpy=3.14159265358979 0.510529087283314 -1.5707963267949
- joint R-FOOT-PITCH: limit lower=-6.28 upper=6.28 effort=80 velocity=15 -> lower=-3.05 upper=1.1 effort=80 velocity=15; origin xyz=-0.0691224724171834 -0.000977844256942021 0.00490279411925121 rpy=0 0.97654912407395 3.14159265358979 -> xyz=-0.071 -0.000977844256941324 0 rpy=0 0.976549124075326 3.14159265358979; type continuous -> revolute
- joint R-FOOT-ROLL: origin xyz=-0.0335980387711934 0 0.00552215574305855 rpy=0 -1.56994489788078 -1.5707963267952 -> xyz=-0.0283480387711934 0 0.00650000000000062 rpy=0 -1.56994489788104 -1.5707963267952; type continuous -> revolute
- joint R-HIP-PITCH: limit lower=-6.28 upper=6.28 effort=80 velocity=15 -> lower=-0.7 upper=3.65 effort=80 velocity=15; origin xyz=-0.0107790968922718 0 -0.0371000000000001 rpy=0 -0.485143684220994 3.14159265358979 -> xyz=-0.00525000000000002 0 0 rpy=0 -0.485143684220995 3.14159265358979; type continuous -> revolute
- joint R-HIP-ROLL: limit lower=-6.28 upper=6.28 effort=80 velocity=15 -> lower=-3.15 upper=1.2 effort=80 velocity=15; origin xyz=-0.00525000000000002 0.0287557819995647 0 rpy=3.14159265358929 1.56467062695372 0 -> xyz=-0.00525000000000004 0.0287557819995579 0 rpy=3.14159265358929 1.56467062695372 0; type continuous -> revolute
- joint R-LINK-ANKLE-TIBIA: origin xyz=0.08225 -0.0165499108803071 0 rpy=1.5707963267949 0 -3.14159265358979 -> xyz=0.08225 -0.00100000000000004 0 rpy=1.5707963267949 0 -3.14159265358979
- joint R-SC-FOOT-PITCH: origin xyz=0 0.01 0 rpy=1.5707963267949 0 -3.14159265358979 -> xyz=0.00525000000000003 0.0101480699951998 0 rpy=1.5707963267949 0 -3.14159265358979
- joint R-SC-HIP-ROLL: origin xyz=0.00995593171266153 -0.038 -0.0083 rpy=1.5707963267949 0 -1.5707963267949 -> xyz=0.00995593171267099 -0.0380000000000001 -0.00829999999999114 rpy=1.5707963267949 0 -1.57079632679491
- joint R-SC2-FOOT-PITCH: origin xyz=0 0 0 rpy=1.5707963267949 0 -3.14159265358979 -> xyz=0.00525000000000005 -0.000977844256941326 0 rpy=1.5707963267949 0 -3.14159265358979
- joint R-SERVO-HIP-PITCH: origin xyz=-2.90968922719282E-05 0.0287557819995648 0.00474991088030713 rpy=1.5707963267949 0 3.14159265358979 -> xyz=0.00549999999999985 -0.00834421800043533 -0.0108 rpy=1.5707963267949 0 3.14159265358979
- joint R-SUCTION: origin xyz=-0.0256224724171834 0 0.00490279411925112 rpy=1.57079632679489 1.42430434544001 0 -> xyz=-0.0275 0 0 rpy=1.57079632679489 1.42430434543863 0; type continuous -> fixed
- joint R-SUCTIONCUP: origin xyz=0 -0.0116636317567742 -0.00454575689710258 rpy=1.06026723948583 0 -3.14159265358979 -> xyz=-0.000701795694196213 -0.00314734742823193 -0.00994844150018426 rpy=0 0 1.57079632679489
- joint R-TIBIA-PITCH: limit lower=-6.28 upper=6.28 effort=80 velocity=15 -> lower=-0.2 upper=3.7 effort=80 velocity=15; origin xyz=0 0 0 rpy=0 1.20507361710935 -3.14159265358979 -> xyz=-0.00525000000000002 0 0 rpy=0 1.20507361711073 -3.14159265358979; type continuous -> revolute
- joint SC-FRONT-CAPLING: origin xyz=0.0471559317126615 0.0105 0.0133 rpy=1.5707963267949 0 0 -> xyz=0.0471559317126484 0.0104999999999991 0.0133000000000366 rpy=1.5707963267949 0 0
- joint SC-REAR-CAPLING: origin xyz=-0.0373440682873384 0.00524999999999999 0.0133 rpy=1.5707963267949 0 -1.5707963267949 -> xyz=-0.0373440682873521 0.00525000000000032 0.0133000000000364 rpy=1.5707963267949 0 -1.57079632679491
