Commit message: digit can stand

File: rsc/digit/digit.urdf (robot description, URDF)
Before this commit: robot digit, 29 links, 28 joints
Joints:
- joint knee_to_shin_left: type fixed -> revolute
- joint knee_to_shin_right: type fixed -> revolute
- joint shoulder_cap_joint_right: type fixed -> revolute
- joint shoulder_roll_cap_left: type fixed -> revolute
- joint waist_cap_joint_left: type fixed -> revolute
- joint waist_cap_joint_right: type fixed -> revolute

Commit message: added leg end effector frames to digit

File: rsc/digit/digit.urdf (robot description, URDF)
Before this commit: robot digit, 29 links, 28 joints
Links:
- added link left_sole
- added link right_sole
Joints:
- added joint LLeg_effector_fixedjoint: type fixed, parent left_toe_roll, child left_sole, origin xyz=0 0 -0.04511 rpy=0 -1.046666667 -1.57079632679, axis 0 0 0
- added joint RLeg_effector_fixedjoint: type fixed, parent right_toe_roll, child right_sole, origin xyz=0 0 -0.04511 rpy=0 -1.046666667 1.57079632679, axis 0 0 0

Commit message: on tuning the gains for digit

File: rsc/digit/digit.urdf (robot description, URDF)
Before this commit: robot digit, 31 links, 30 joints
Joints:
- joint LLeg_effector_fixedjoint: origin xyz=0 0 -0.04511 rpy=0 -1.046666667 -1.57079632679 -> xyz=0 -0.052545 -0.030374 rpy=0 -1.046666667 -1.57079632679
- joint RLeg_effector_fixedjoint: origin xyz=0 0 -0.04511 rpy=0 -1.046666667 1.57079632679 -> xyz=0 0.052545 -0.030374 rpy=0 -1.046666667 1.57079632679

Commit message: on PD gains for Digit

File: rsc/digit/digit.urdf (robot description, URDF)
Before this commit: robot digit, 31 links, 30 joints
Links:
- link left_elbow: geometry visual mesh filename=meshes/arm-L4.obj
- link left_hip_pitch: geometry visual mesh filename=meshes/hip-pitch.obj
- link left_hip_roll: geometry visual mesh filename=meshes/hip-yaw-housing.obj
- link left_hip_yaw: geometry visual mesh filename=meshes/hip-pitch-housing.obj
- link left_knee: geometry visual mesh filename=meshes/knee.obj
- link left_shin: geometry visual mesh filename=meshes/shin.obj
- link left_shoulder_cap: geometry visual mesh filename=meshes/shoulder-roll-housing.obj
- link left_shoulder_pitch: geometry visual mesh filename=meshes/arm-L2.obj
- link left_shoulder_roll: geometry visual mesh filename=meshes/arm-L1.obj
- link left_shoulder_yaw: geometry visual mesh filename=meshes/arm-L3.obj
- link left_tarsus: geometry visual mesh filename=meshes/tarsus.obj
- link left_waist_cap: geometry visual mesh filename=meshes/shoulder-roll-housing.obj
- link right_elbow: geometry visual mesh filename=meshes/arm-L4.obj scale=1 -1 1
- link right_hip_pitch: geometry visual mesh filename=meshes/hip-pitch.obj scale=1 -1 1
- link right_hip_roll: geometry visual mesh filename=meshes/hip-yaw-housing.obj scale=1 -1 1
- link right_hip_yaw: geometry visual mesh filename=meshes/hip-pitch-housing.obj scale=1 -1 1
- link right_knee: geometry visual mesh filename=meshes/knee.obj scale=1 -1 1
- link right_shin: geometry visual mesh filename=meshes/shin.obj scale=1 -1 1
- link right_shoulder_cap: geometry visual mesh filename=meshes/shoulder-roll-housing.obj scale=1 -1 1
- link right_shoulder_pitch: geometry visual mesh filename=meshes/arm-L2.obj scale=1 -1 1
- link right_shoulder_roll: geometry visual mesh filename=meshes/arm-L1.obj scale=1 -1 1
- link right_shoulder_yaw: geometry visual mesh filename=meshes/arm-L3.obj scale=1 -1 1
- link right_tarsus: geometry visual mesh filename=meshes/tarsus.obj scale=1 -1 1
- link right_waist_cap: geometry visual mesh filename=meshes/shoulder-roll-housing.obj scale=1 -1 1
- link torso: geometry visual mesh filename=meshes/torso.obj
Joints:
- joint knee_to_shin_left: type revolute -> fixed
- joint knee_to_shin_right: type revolute -> fixed
- joint shoulder_cap_joint_right: type revolute -> fixed
- joint shoulder_roll_cap_left: type revolute -> fixed
- joint waist_cap_joint_left: type revolute -> fixed
- joint waist_cap_joint_right: type revolute -> fixed
